File: MBI5024.kicad_pcb (KiCad board)
At the start: 2 copper layers, 31.5 x 21.8 mm, 3 parts, among them J1 Conn_01x12, J2 Conn_01x12, U1 MBI5024

Commit message: Fixed up PCB
Parts:
- J2: value Conn_01x12 -> Conn_01x12_13-24; footprint Connector_PinHeader_2.54mm:PinHeader_1x12_P2.54mm_Vertical -> Connectors:PinHeader_1x12_P2.54mm_Vertical_13-24
- moved J1 28.2 mm to (122.9, 101.6), turned to 270 degrees
- moved J2 27.9 mm to (151.1, 83.3), turned to 90 degrees
Connections:
- U1 pad 1: Net-(J1-Pad12) -> Net-(J1-Pad1)
- U1 pad 10: Net-(J1-Pad3) -> Net-(J1-Pad10)
- U1 pad 11: Net-(J1-Pad2) -> Net-(J1-Pad11)
- U1 pad 12: Net-(J1-Pad1) -> Net-(J1-Pad12)
- U1 pad 13: Net-(J2-Pad12) -> Net-(J2-Pad13)
- U1 pad 14: Net-(J2-Pad11) -> Net-(J2-Pad14)
- U1 pad 15: Net-(J2-Pad10) -> Net-(J2-Pad15)
- U1 pad 16: Net-(J2-Pad9) -> Net-(J2-Pad16)
- U1 pad 17: Net-(J2-Pad8) -> Net-(J2-Pad17)
- U1 pad 18: Net-(J2-Pad7) -> Net-(J2-Pad18)
- U1 pad 19: Net-(J2-Pad6) -> Net-(J2-Pad19)
- U1 pad 2: Net-(J1-Pad11) -> Net-(J1-Pad2)
- U1 pad 20: Net-(J2-Pad5) -> Net-(J2-Pad20)
- U1 pad 21: Net-(J2-Pad4) -> Net-(J2-Pad21)
- U1 pad 22: Net-(J2-Pad3) -> Net-(J2-Pad22)
- U1 pad 23: Net-(J2-Pad2) -> Net-(J2-Pad23)
- U1 pad 24: Net-(J2-Pad1) -> Net-(J2-Pad24)
- U1 pad 3: Net-(J1-Pad10) -> Net-(J1-Pad3)
- U1 pad 4: Net-(J1-Pad9) -> Net-(J1-Pad4)
- U1 pad 5: Net-(J1-Pad8) -> Net-(J1-Pad5)
- U1 pad 6: Net-(J1-Pad7) -> Net-(J1-Pad6)
- U1 pad 7: Net-(J1-Pad6) -> Net-(J1-Pad7)
- U1 pad 8: Net-(J1-Pad5) -> Net-(J1-Pad8)
- U1 pad 9: Net-(J1-Pad4) -> Net-(J1-Pad9)
Routing:
- net Net-(J2-Pad24): track 0.00 -> 10.8 mm
- net Net-(J2-Pad13): track 0.00 -> 10.8 mm
- net Net-(J2-Pad12): track 10.8 -> 0.00 mm
- net Net-(J2-Pad1): track 10.8 -> 0.00 mm
- net Net-(J2-Pad23): track 0.00 -> 10.2 mm
- net Net-(J2-Pad14): track 0.00 -> 10.1 mm
- net Net-(J2-Pad11): track 10.1 -> 0.00 mm
- net Net-(J2-Pad2): track 10.1 -> 0.00 mm
- net Net-(J2-Pad15): track 0.00 -> 9.31 mm
- net Net-(J2-Pad10): track 9.31 -> 0.00 mm
- net Net-(J2-Pad3): track 9.31 -> 0.00 mm
- net Net-(J2-Pad22): track 0.00 -> 9.31 mm
- net Net-(J2-Pad21): track 0.00 -> 8.03 mm
- net Net-(J2-Pad9): track 7.93 -> 0.00 mm
- net Net-(J2-Pad4): track 7.93 -> 0.00 mm
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