File: MBI5024_Adapter.sch (KiCad schematic (older format))
At the start: 3 parts, among them J1 Conn_01x12, J2 Conn_01x12_13-24, U1 MBI5024

Commit message: Renamed project
Parts:
- U1: footprint MBI5024_Footprint_Library:SSOP-24-1mm -> MBI5024:SSOP-24-1mm
Changed lines of the file:
@@
 EESchema Schematic File Version 4
-LIBS:MBI5024-cache
 EELAYER 26 0
 EELAYER END
@@
 F 0 "U1" H 5150 4450 50  0000 C CNN
 F 1 "MBI5024" H 5750 2600 50  0000 C CNN
-F 2 "MBI5024_Footprint_Library:SSOP-24-1mm" H 5550 3800 50  0001 C CNN
+F 2 "MBI5024:SSOP-24-1mm" H 5550 3800 50  0001 C CNN
 F 3 "" H 5550 3800 50  0001 C CNN
 	1    5500 3600
