File: MBI5024_Adapter.kicad_pcb (KiCad board)
At the start: 2 copper layers, 31.5 x 21.8 mm, 3 parts, among them J1 Conn_01x12, J2 Conn_01x12_13-24, U1 MBI5024

Commit message: Generate new pcb to make sure the pipeline works
Parts:
- U1: footprint MBI5024_Footprint_Library:SSOP-24-1mm -> MBI5024:SSOP-24-1mm
